File: 4ch-relay-pcb.kicad_pcb (KiCad board)
At the start: 2 copper layers, 41 parts, among them J1 Screw_Terminal_01x03, J2 Conn_01x06_Pin, J3 Screw_Terminal_01x03, J4 Screw_Terminal_01x03, J5 Screw_Terminal_01x03, K1 Relay_SPDT, K2 Relay_SPDT, K3 Relay_SPDT, K4 Relay_SPDT, Q1 2N3904, Q2 2N3904, Q3 2N3904, Q4 2N3904, U1 PC817, U2 PC817, U3 PC817, U4 PC817

Commit message: Add files via upload
Other:
- board text added: "5v"
- board text added: "G"
- board text added: "R1"
- board text added: "R2"
- board text added: "R3"
- board text added: "R4"
Changed lines of the file:
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@@
 		)
+	)
+	(gr_poly
+		(pts
+			(xy 134.24 64.44) (xy 136.27 64.45) (xy 136.27 87.1) (xy 134.25 87.09) (xy 134.25 64.43)
+		)
+		(stroke
+			(width 0.1)
+			(type solid)
+		)
+		(fill yes)
+		(layer "B.Mask")
+	)
+	(gr_poly
+		(pts
+			(xy 112.93 64.36) (xy 112.93 87.22) (xy 112.35 86.9) (xy 111.82 86.62) (xy 111.31 86.71) (xy 111.17 86.97)
+			(xy 111.03 87.19) (xy 110.93 87.25) (xy 110.92 87.22) (xy 110.91 87.16) (xy 110.91 64.36)
+		)
+		(stroke
+			(width 0.1)
+			(type solid)
+		)
+		(fill yes)
+		(layer "B.Mask")
+	)
+	(gr_poly
+		(pts
+			(xy 159.18 64.37) (xy 159.17 87.01) (xy 158.87 86.84) (xy 158.25 86.65) (xy 157.93 86.69) (xy 157.77 86.78)
+			(xy 157.53 86.91) (xy 157.42 87.06) (xy 157.18 87.3) (xy 157.17 87.23) (xy 157.17 64.37)
+		)
+		(stroke
+			(width 0.1)
+			(type solid)
+		)
+		(fill yes)
+		(layer "B.Mask")
+	)
+	(gr_poly
+		(pts
+			(xy 107.860453 64.32) (xy 107.86 72.87) (xy 107.777335 73.121108) (xy 107.66 73.3) (xy 107.5 73.46)
+			(xy 107.28 73.66) (xy 107.09 73.84) (xy 106.91 73.11) (xy 106.68 72.75) (xy 106.27 72.52) (xy 105.8 72.46)
+			(xy 105.62 72.46) (xy 105.68 72.35) (xy 105.82 72.22) (xy 105.82 64.32)
+		)
+		(stroke
+			(width 0.1)
+			(type solid)
+		)
+		(fill yes)
+		(layer "B.Mask")
+	)
+	(gr_poly
+		(pts
+			(xy 182.59 64.37) (xy 182.59 86.98) (xy 182.5 86.9) (xy 182.35 86.78) (xy 182.17 86.68) (xy 181.93 86.59)
+			(xy 181.7 86.57) (xy 181.49 86.58) (xy 181.37 86.6) (xy 181.13 86.71) (xy 180.9 86.87) (xy 180.76 87.02)
+			(xy 180.62 87.24) (xy 180.58 87.32) (xy 180.58 64.37)
+		)
+		(stroke
+			(width 0.1)
+			(type solid)
+		)
+		(fill yes)
+		(layer "B.Mask")
+	)
+	(gr_poly
+		(pts
+			(xy 141.36 64.9) (xy 141.36 72.22) (xy 141.55 72.41) (xy 141.03 72.42) (xy 140.7 72.55) (xy 140.46 72.75)
+			(xy 140.25 73.01) (xy 140.19 73.24) (xy 140.16 73.36) (xy 140.15 73.7) (xy 140.13 73.82) (xy 140.07 73.8)
+			(xy 139.68 73.41) (xy 139.55 73.29) (xy 139.47 73.17) (xy 139.38 73.02) (xy 139.33 72.8) (xy 139.32 72.65)
+			(xy 139.32 64.9)
+		)
+		(stroke
+			(width 0.1)
+			(type solid)
+		)
+		(fill yes)
+		(layer "B.Mask")
+	)
+	(gr_poly
+		(pts
+			(xy 115.99 64.83) (xy 118.01 64.83) (xy 118.01 72.2) (xy 118.2 72.39) (xy 118.15 72.4) (xy 117.83 72.39)
+			(xy 117.51 72.47) (xy 117.25 72.61) (xy 116.99 72.86) (xy 116.85 73.14) (xy 116.78 73.47) (xy 116.79 73.8)
+			(xy 116.76 73.8) (xy 116.26 73.3) (xy 116.2 73.23) (xy 116.16 73.17) (xy 116.12 73.1) (xy 116.08 73.02)
+			(xy 116.04 72.93) (xy 116 72.78) (xy 115.99 72.63)
+		)
+		(stroke
+			(width 0.1)
+			(type solid)
+		)
+		(fill yes)
+		(layer "B.Mask")
+	)
+	(gr_poly
+		(pts
+			(xy 129.17 64.45) (xy 131.18 64.45) (xy 131.18 72.67) (xy 131.17 72.78) (xy 131.15 72.86) (xy 131.12 72.96)
+			(xy 131.09 73.04) (xy 131.02 73.17) (xy 130.97 73.24) (xy 130.89 73.33) (xy 130.42 73.8) (xy 130.42 73.56)
+			(xy 130.39 73.31) (xy 130.33 73.14) (xy 130.22 72.94) (xy 129.94 72.64) (xy 129.68 72.5) (xy 129.4 72.42)
+			(xy 129.11 72.38) (xy 129.01 72.37) (xy 129.17 72.21)
+		)
+		(stroke
+			(width 0.1)
+			(type solid)
+		)
+		(fill yes)
+		(layer "B.Mask")
 	)
 	(gr_rect
@@
 			)
 			(justify left bottom)
+		)
+	)
+	(gr_text "5v"
+		(at 135.13 127.36 0)
+		(layer "F.Fab")
+		(effects
+			(font
+				(size 1 1)
+				(thickness 0.15)
+			)
+			(justify left bottom)
+		)
+	)
+	(gr_text "G"
+		(at 138.1 127.36 0)
+		(layer "F.Fab")
+		(effects
+			(font
+				(size 1 1)
+				(thickness 0.15)
+			)
+			(justify left bottom)
+		)
+	)
+	(gr_text "R1"
+		(at 140.25 127.36 0)
+		(layer "F.Fab")
+		(effects
+			(font
+				(size 1 1)
+				(thickness 0.15)
+			)
+			(justify left bottom)
+		)
+	)
+	(gr_text "R2"
+		(at 142.67 127.37 0)
+		(layer "F.Fab")
+		(effects
+			(font
+				(size 1 1)
+				(thickness 0.15)
+			)
+			(justify left bottom)
+		)
+	)
+	(gr_text "R3"
+		(at 145.15 127.38 0)
+		(layer "F.Fab")
+		(effects
+			(font
+				(size 1 1)
+				(thickness 0.15)
+			)
+			(justify left bottom)
+		)
+	)
+	(gr_text "R4"
+		(at 147.8 127.38 0)
+		(layer "F.Fab")
+		(effects
+			(font
+				(size 1 1)
+				(thickness 0.15)
+			)
+			(justify left bottom)
