File: 4ch-relay-pcb.kicad_pcb (KiCad board)
At the start: 2 copper layers, 41 parts, among them J1 Screw_Terminal_01x03, J2 Conn_01x06_Pin, J3 Screw_Terminal_01x03, J4 Screw_Terminal_01x03, J5 Screw_Terminal_01x03, K1 Relay_SPDT, K2 Relay_SPDT, K3 Relay_SPDT, K4 Relay_SPDT, Q1 2N3904, Q2 2N3904, Q3 2N3904, Q4 2N3904, U1 PC817, U2 PC817, U3 PC817, U4 PC817

Commit message: Add files via upload
Other:
- board outline added: 98.2 x 76.4 mm
- board text added: "CO"
- board text added: "NC"
- board text added: "NO"
Changed lines of the file:
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@@
 		(layer "F.SilkS")
+	)
+	(gr_rect
+		(start 97.42 54.29)
+		(end 195.58 130.7)
+		(stroke
+			(width 0.05)
+			(type default)
+		)
+		(fill no)
+		(layer "Edge.Cuts")
 	)
 	(gr_text "SASoftwareS"
@@
 		)
 	)
+	(gr_text "NC"
+		(at 107.07 57.14 90)
+		(layer "F.SilkS")
+		(effects
+			(font
+				(size 0.8 0.8)
+				(thickness 0.1)
+			)
+			(justify left bottom)
+		)
+	)
+	(gr_text "CO"
+		(at 112.29 57.11 90)
+		(layer "F.SilkS")
+		(effects
+			(font
+				(size 0.8 0.8)
+				(thickness 0.1)
+			)
+			(justify left bottom)
+		)
+	)
+	(gr_text "NO"
+		(at 117.14 57.14 90)
+		(layer "F.SilkS")
+		(effects
+			(font
+				(size 0.8 0.8)
+				(thickness 0.1)
+			)
+			(justify left bottom)
+		)
+	)
+	(gr_text "NC"
+		(at 130.41 57.31 90)
+		(layer "F.SilkS")
+		(effects
+			(font
+				(size 0.8 0.8)
+				(thickness 0.1)
+			)
+			(justify left bottom)
+		)
+	)
+	(gr_text "CO"
+		(at 135.63 57.28 90)
+		(layer "F.SilkS")
+		(effects
+			(font
+				(size 0.8 0.8)
+				(thickness 0.1)
+			)
+			(justify left bottom)
+		)
+	)
+	(gr_text "NO"
+		(at 140.48 57.31 90)
+		(layer "F.SilkS")
+		(effects
+			(font
+				(size 0.8 0.8)
+				(thickness 0.1)
+			)
+			(justify left bottom)
+		)
+	)
+	(gr_text "NC"
+		(at 153.16 57.26 90)
+		(layer "F.SilkS")
+		(effects
+			(font
+				(size 0.8 0.8)
+				(thickness 0.1)
+			)
+			(justify left bottom)
+		)
+	)
+	(gr_text "CO"
+		(at 158.38 57.23 90)
+		(layer "F.SilkS")
+		(effects
+			(font
+				(size 0.8 0.8)
+				(thickness 0.1)
+			)
+			(justify left bottom)
+		)
+	)
+	(gr_text "NO"
+		(at 163.23 57.26 90)
+		(layer "F.SilkS")
+		(effects
+			(font
+				(size 0.8 0.8)
+				(thickness 0.1)
+			)
+			(justify left bottom)
+		)
+	)
+	(gr_text "NC"
+		(at 176.5 57.29 90)
+		(layer "F.SilkS")
+		(effects
+			(font
+				(size 0.8 0.8)
+				(thickness 0.1)
+			)
+			(justify left bottom)
+		)
+	)
+	(gr_text "CO"
+		(at 181.72 57.26 90)
+		(layer "F.SilkS")
+		(effects
+			(font
+				(size 0.8 0.8)
+				(thickness 0.1)
+			)
+			(justify left bottom)
+		)
+	)
+	(gr_text "NO"
+		(at 186.57 57.29 90)
+		(layer "F.SilkS")
+		(effects
+			(font
+				(size 0.8 0.8)
+				(thickness 0.1)
+			)
+			(justify left bottom)
+		)
+	)

Commit message: Add files via upload
Parts:
- added ?: , , F.Cu at (192.5, 57.4)
- added ?: , , F.Cu at (191.9, 127.0)
- added ?: , , F.Cu at (100.6, 57.5)
- added ?: , , F.Cu at (101.0, 127.1)
Other:
- board text added: "5v G R1 R2 R3 R4"
- board text removed: "5v"
- board text removed: "G"
- board text removed: "R1"
- board text removed: "R2"
- board text removed: "R3"
- board text removed: "R4"
